File: 5vCharger.sch (KiCad schematic (older format))
At the start: 12 parts, among them J1 Screw_Terminal_1x02, U1 LM2596

Commit message: calculated and put values of components
Parts:
- added C1, C5: 100n, symbol C
- added LED1: LED, symbol LED
- added R4: 1k, symbol R
- added ZD1: 5v1, symbol D_Zener
- C2: renamed from C?; value CP1 -> 220u
- C3: renamed from C?; value CP1 -> 470u
- C4: renamed from C?; value C -> 10n
- D1: renamed from D?; value D_Schottky -> 1N5822
- L1: renamed from L?; value L -> 22u
- R1: renamed from R?; value R -> 10k
- R2: renamed from R?; value R -> 1k
- R3: renamed from R?; value R -> 3k
- gave numbers to parts that had none: 2
Connections:
- net at C2.1, J1.1, R1.1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: now also C1.1
- net at C2.2, C3.2, D1.2 (A)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: now also C1.2, C5.2, LED1.1 (K), ZD1.2 (A)
- net at R1.2, SW1.1 (P1), U1.5 (~On~/Off): now also ZD1.1 (K)
- net at C3.1, J2.1, L1.2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: now also C4.1, C5.1, R4.1
- new net: LED1.2 (A), R4.2
Other:
- note added: "Switch Contacts"
- moved on the sheet: J1, J2
Changed lines of the file:
@@
 L Screw_Terminal_1x02 J1
 U 1 1 598C0486
-P 4050 3550
-F 0 "J1" H 4050 3800 50  0000 C TNN
-F 1 "Screw_Terminal_1x02" V 3900 3550 50  0000 C TNN
-F 2 "" H 4050 3325 50  0001 C CNN
-F 3 "" H 4025 3550 50  0001 C CNN
-	1    4050 3550
-	1    0    0    -1
-$EndComp
-Wire Wire Line
-	4250 3450 4900 3450
-$Comp
-L CP1 C?
+P 3800 3550
+F 0 "J1" H 3800 3800 50  0000 C TNN
+F 1 "Screw_Terminal_1x02" V 3650 3550 50  0000 C TNN
+F 2 "" H 3800 3325 50  0001 C CNN
+F 3 "" H 3775 3550 50  0001 C CNN
+	1    3800 3550
+	1    0    0    -1
+$EndComp
+Wire Wire Line
+	4000 3450 4250 3450
+Wire Wire Line
+	4250 3450 4600 3450
+Wire Wire Line
+	4600 3450 4900 3450
+$Comp
+L CP1 C2
 U 1 1 598C050C
 P 4600 4000
-F 0 "C?" H 4625 4100 50  0000 L CNN
-F 1 "CP1" H 4625 3900 50  0000 L CNN
+F 0 "C2" H 4625 4100 50  0000 L CNN
+F 1 "220u" H 4625 3900 50  0000 L CNN
 F 2 "" H 4600 4000 50  0000 C CNN
 F 3 "" H 4600 4000 50  0000 C CNN
@@
 Connection ~ 4600 3450
 Wire Wire Line
-	4250 3650 4250 4450
-Wire Wire Line
-	4250 4450 8050 4450
+	4000 3650 4000 4450
+Wire Wire Line
+	4000 4450 4250 4450
+Wire Wire Line
+	4250 4450 4600 4450
+Wire Wire Line
+	4600 4450 4900 4450
+Wire Wire Line
+	4900 4450 5400 4450
+Wire Wire Line
+	5400 4450 5850 4450
+Wire Wire Line
+	5850 4450 6400 4450
+Wire Wire Line
+	6400 4450 6700 4450
+Wire Wire Line
+	6700 4450 7350 4450
+Wire Wire Line
+	7350 4450 8050 4450
+Wire Wire Line
+	8050 4450 8300 4450
+Wire Wire Line
+	8300 4450 8550 4450
 Wire Wire Line
 	5400 4150 5400 4450
@@
 Wire Wire Line
 	4600 4150 4600 4450
-Wire Wire Line
-	4600 4450 4550 4450
-Connection ~ 4550 4450
-$Comp
-L R R?
+$Comp
+L R R1
 U 1 1 598C05E8
 P 4900 3600
-F 0 "R?" V 4980 3600 50  0000 C CNN
-F 1 "R" V 4900 3600 50  0000 C CNN
+F 0 "R1" V 4980 3600 50  0000 C CNN
+F 1 "10k" V 4900 3600 50  0000 C CNN
 F 2 "" V 4830 3600 50  0000 C CNN
 F 3 "" H 4900 3600 50  0000 C CNN
@@
 	4900 4150 5850 4150
 $Comp
-L CONN_01X02 P?
+L CONN_01X02 SW1
 U 1 1 598C0644
 P 6050 4300
-F 0 "P?" H 6050 4450 50  0000 C CNN
+F 0 "SW1" H 6050 4450 50  0000 C CNN
 F 1 "CONN_01X02" V 6150 4300 50  0000 C CNN
 F 2 "" H 6050 4300 50  0000 C CNN
@@
 Connection ~ 5850 4450
 $Comp
-L CP1 C?
+L CP1 C3
 U 1 1 598C0736
 P 7350 4000
-F 0 "C?" H 7375 4100 50  0000 L CNN
-F 1 "CP1" H 7375 3900 50  0000 L CNN
+F 0 "C3" H 7375 4100 50  0000 L CNN
+F 1 "470u" H 7375 3900 50  0000 L CNN
 F 2 "" H 7350 4000 50  0000 C CNN
 F 3 "" H 7350 4000 50  0000 C CNN
@@
 $EndComp
 $Comp
-L D_Schottky D?
+L D_Schottky D1
 U 1 1 598C0783
 P 6700 4000
-F 0 "D?" H 6700 4100 50  0000 C CNN
-F 1 "D_Schottky" H 6700 3900 50  0000 C CNN
+F 0 "D1" H 6700 4100 50  0000 C CNN
+F 1 "1N5822" H 6700 3900 50  0000 C CNN
 F 2 "" H 6700 4000 50  0000 C CNN
 F 3 "" H 6700 4000 50  0000 C CNN
@@
 $EndComp
 $Comp
-L L L?
+L L L1
 U 1 1 598C07E4
 P 7000 3400
-F 0 "L?" V 6950 3400 50  0000 C CNN
-F 1 "L" V 7075 3400 50  0000 C CNN
+F 0 "L1" V 6950 3400 50  0000 C CNN
+F 1 "22u" V 7075 3400 50  0000 C CNN
 F 2 "" H 7000 3400 50  0000 C CNN
 F 3 "" H 7000 3400 50  0000 C CNN
@@
 Connection ~ 6700 4450
 $Comp
-L R R?
+L R R3
 U 1 1 598C08D3
 P 7550 3550
-F 0 "R?" V 7630 3550 50  0000 C CNN
-F 1 "R" V 7550 3550 50  0000 C CNN
+F 0 "R3" V 7630 3550 50  0000 C CNN
+F 1 "3k" V 7550 3550 50  0000 C CNN
 F 2 "" V 7480 3550 50  0000 C CNN
 F 3 "" H 7550 3550 50  0000 C CNN
@@
 	6400 3450 6400 3400
 Wire Wire Line
-	6400 3400 6850 3400
-Wire Wire Line
-	7150 3400 8050 3400
-Wire Wire Line
-	6400 3700 7800 3700
+	6400 3400 6700 3400
+Wire Wire Line
+	6700 3400 6850 3400
+Wire Wire Line
+	7150 3400 7350 3400
+Wire Wire Line
+	7350 3400 7550 3400
+Wire Wire Line
+	7550 3400 7800 3400
+Wire Wire Line
+	7800 3400 8050 3400
+Wire Wire Line
+	8050 3400 8300 3400
+Wire Wire Line
+	8300 3400 8550 3400
+Wire Wire Line
+	6400 3700 7550 3700
 Connection ~ 7350 3400
 $Comp
-L R R?
+L R R2
 U 1 1 598C0B73
 P 6400 4050
-F 0 "R?" V 6480 4050 50  0000 C CNN
-F 1 "R" V 6400 4050 50  0000 C CNN
+F 0 "R2" V 6480 4050 50  0000 C CNN
+F 1 "1k" V 6400 4050 50  0000 C CNN
 F 2 "" V 6330 4050 50  0000 C CNN
 F 3 "" H 6400 4050 50  0000 C CNN
@@
 Connection ~ 6400 4450
 Connection ~ 7550 3400
-$Comp
-L C C?
+Connection ~ 7550 3700
+$Comp
+L Screw_Terminal_1x02 J2
+U 1 1 598C0DCE
+P 8750 3950
+F 0 "J2" H 8750 4200 50  0000 C TNN
+F 1 "Screw_Terminal_1x02" V 8600 3950 50  0000 C TNN
+F 2 "" H 8750 3725 50  0001 C CNN
+F 3 "" H 8725 3950 50  0001 C CNN
+	1    8750 3950
+	-1   0    0    -1
+$EndComp
+Wire Wire Line
+	8550 3400 8550 3850
+Wire Wire Line
+	8550 4450 8550 4050
+$Comp
+L LED LED1
+U 1 1 598C2A6C
+P 8300 4150
+F 0 "LED1" H 8300 4250 50  0000 C CNN
+F 1 "LED" H 8300 4050 50  0000 C CNN
+F 2 "" H 8300 4150 50  0000 C CNN
+F 3 "" H 8300 4150 50  0000 C CNN
+	1    8300 4150
+	0    -1   -1   0
+$EndComp
+$Comp
+L R R4
+U 1 1 598C2B30
+P 8300 3700
+F 0 "R4" V 8380 3700 50  0000 C CNN
+F 1 "1k" V 8300 3700 50  0000 C CNN
+F 2 "" V 8230 3700 50  0000 C CNN
+F 3 "" H 8300 3700 50  0000 C CNN
+	1    8300 3700
+	1    0    0    -1
+$EndComp
+Wire Wire Line
+	8300 3400 8300 3550
+Connection ~ 8050 3400
+Wire Wire Line
+	8300 3850 8300 4000
+Wire Wire Line
+	8300 4450 8300 4300
+Connection ~ 8050 4450
+Connection ~ 4600 4450
+$Comp
+L C C1
+U 1 1 598C2EA0
+P 4250 4000
+F 0 "C1" H 4275 4100 50  0000 L CNN
+F 1 "100n" H 4275 3900 50  0000 L CNN
+F 2 "" H 4288 3850 50  0000 C CNN
+F 3 "" H 4250 4000 50  0000 C CNN
+	1    4250 4000
+	1    0    0    -1
+$EndComp
+Wire Wire Line
+	4250 3850 4250 3450
+Connection ~ 4250 3450
+Wire Wire Line
+	4250 4150 4250 4450
+Connection ~ 4250 4450
+Connection ~ 8300 3400
+Connection ~ 8300 4450
+$Comp
+L C C5
+U 1 1 598C3227
+P 8050 4000
+F 0 "C5" H 8075 4100 50  0000 L CNN
+F 1 "100n" H 8075 3900 50  0000 L CNN
+F 2 "" H 8088 3850 50  0000 C CNN
+F 3 "" H 8050 4000 50  0000 C CNN
+	1    8050 4000
+	-1   0    0    -1
+$EndComp
+Wire Wire Line
+	8050 3850 8050 3400
+Wire Wire Line
+	8050 4150 8050 4450
+Text Notes 5700 4700 0    60   ~ 0
+Switch Contacts
+Connection ~ 5850 4150
+Connection ~ 4900 3450
+Connection ~ 6400 3700
+Connection ~ 7800 3400
+$Comp
+L D_Zener ZD1
+U 1 1 598C3D71
+P 4900 4300
+F 0 "ZD1" H 4900 4400 50  0000 C CNN
+F 1 "5v1" H 4900 4200 50  0000 C CNN
+F 2 "" H 4900 4300 50  0000 C CNN
+F 3 "" H 4900 4300 50  0000 C CNN
+	1    4900 4300
+	0    1    1    0
+$EndComp
+Connection ~ 4900 4450
+$Comp
+L C C4
 U 1 1 598C0CD0
 P 7800 3550
-F 0 "C?" H 7825 3650 50  0000 L CNN
-F 1 "C" H 7825 3450 50  0000 L CNN
+F 0 "C4" H 7825 3650 50  0000 L CNN
+F 1 "10n" H 7825 3450 50  0000 L CNN
 F 2 "" H 7838 3400 50  0000 C CNN
 F 3 "" H 7800 3550 50  0000 C CNN
@@
 	1    0    0    -1
 $EndComp
-Connection ~ 7550 3700
-$Comp
-L Screw_Terminal_1x02 J?
-U 1 1 598C0DCE
-P 8250 3950
-F 0 "J?" H 8250 4200 50  0000 C TNN
-F 1 "Screw_Terminal_1x02" V 8100 3950 50  0000 C TNN
-F 2 "" H 8250 3725 50  0001 C CNN
-F 3 "" H 8225 3950 50  0001 C CNN
-	1    8250 3950
-	-1   0    0    -1
-$EndComp
-Wire Wire Line
-	8050 3400 8050 3850
-Wire Wire Line
-	8050 4450 8050 4050
+Wire Wire Line
+	7550 3700 7800 3700
 $EndSCHEMATC
